File: Payload2020_SIPM_board/Payload2020_SIPM_board.kicad_pcb (KiCad board)
At the start: 2 copper layers, 25 x 25 mm, 13 parts, among them J1 Conn_01x03, U3 TLV2402-Q1, U4 TLV2402-Q1

Commit message: Fixed small errors from last commit
Parts:
- added U2: Broadcom_sipm, Payload2020_custom:Broadcom_SiPM_Breakout, B.Cu at (72.5, 81.8)
Changed lines of the file:
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@@
     (tracks 103)
     (zones 0)
-    (modules 13)
-    (nets 9)
+    (modules 14)
+    (nets 10)
   )
   (page A4)
@@
     (32 B.Adhes user)
     (33 F.Adhes user)
-    (34 B.Paste user hide)
+    (34 B.Paste user)
     (35 F.Paste user)
     (36 B.SilkS user)
     (37 F.SilkS user)
-    (38 B.Mask user hide)
-    (39 F.Mask user hide)
+    (38 B.Mask user)
+    (39 F.Mask user)
     (40 Dwgs.User user hide)
     (41 Cmts.User user hide)
@@
   (net 7 "Net-(D1-Pad1)")
   (net 8 "Net-(R5-Pad1)")
+  (net 9 "Net-(C6-Pad1)")
   (net_class Default "This is the default net class."
     (clearance 0.2)
@@
     (add_net GND)
     (add_net "Net-(C12-Pad1)")
+    (add_net "Net-(C6-Pad1)")
     (add_net "Net-(C9-Pad1)")
     (add_net "Net-(C9-Pad2)")
@@
     (add_net "Net-(R5-Pad1)")
   )
+  (module Payload2020_custom:Broadcom_SiPM_Breakout (layer B.Cu)
+    (at 72.5 81.8 90)
+    (fp_text reference U2 (at -0.9 -8.6 90) (layer B.SilkS)
+      (effects (font (size 1 1) (thickness 0.15)) (justify mirror))
+    )
+    (fp_text value Broadcom_sipm (at 9.1 -2.2) (layer B.Fab)
+      (effects (font (size 1 1) (thickness 0.15)) (justify mirror))
+    )
+    (fp_arc (start 2.65 -1.8) (end 3.149999 -0.750001) (angle 239.1534439) (layer B.SilkS) (width 0.12))
+    (fp_line (start 2.1 1.05) (end 2.85 1.05) (layer B.SilkS) (width 0.12))
+    (fp_line (start 2.5 2.2) (end 3.3 0.05) (layer B.SilkS) (width 0.12))
+    (fp_line (start 1.75 0) (end 2.5 2.2) (layer B.SilkS) (width 0.12))
+    (fp_line (start 4.55 -3.15) (end 4.55 -0.45) (layer B.SilkS) (width 0.12))
+    (fp_line (start 4.55 -3.15) (end 5.9 -3.15) (layer B.SilkS) (width 0.12))
+    (fp_line (start 7.2 -3.15) (end 7.2 -0.45) (layer B.SilkS) (width 0.12))
+    (fp_line (start 7.2 -0.45) (end 7.2 2.25) (layer B.SilkS) (width 0.12))
+    (fp_line (start 4.55 2.25) (end 7.2 2.25) (layer B.SilkS) (width 0.12))
+    (fp_line (start 7.2 -0.45) (end 4.55 -0.45) (layer B.SilkS) (width 0.12))
+    (fp_circle (center 5.9 0.9) (end 6.65 0.65) (layer B.SilkS) (width 0.12))
+    (fp_line (start 7.2 -3.15) (end 4.55 -3.15) (layer B.SilkS) (width 0.12))
+    (fp_line (start 4.55 -0.45) (end 7.2 -0.45) (layer B.SilkS) (width 0.12))
+    (fp_circle (center 5.9 -1.8) (end 6.65 -2.05) (layer B.SilkS) (width 0.12))
+    (fp_line (start 4.55 -0.45) (end 5.9 -0.45) (layer B.SilkS) (width 0.12))
+    (fp_line (start 4.55 -0.45) (end 4.55 2.25) (layer B.SilkS) (width 0.12))
+    (fp_line (start 8 2.25) (end 8 3.2) (layer B.SilkS) (width 0.12))
+    (fp_line (start -7.25 -1.5) (end -4.6 -1.5) (layer B.SilkS) (width 0.12))
+    (fp_line (start -4.6 -4.2) (end -4.6 -1.5) (layer B.SilkS) (width 0.12))
+    (fp_line (start -4.6 -4.2) (end -7.25 -4.2) (layer B.SilkS) (width 0.12))
+    (fp_line (start -7.25 -4.2) (end -7.25 -1.5) (layer B.SilkS) (width 0.12))
+    (fp_line (start -7.25 -4.2) (end -5.9 -4.2) (layer B.SilkS) (width 0.12))
+    (fp_line (start -4.6 -6.9) (end -4.6 -4.2) (layer B.SilkS) (width 0.12))
+    (fp_line (start -7.25 -6.9) (end -5.9 -6.9) (layer B.SilkS) (width 0.12))
+    (fp_line (start -7.25 -4.2) (end -4.6 -4.2) (layer B.SilkS) (width 0.12))
+    (fp_line (start -7.25 -6.9) (end -7.25 -4.2) (layer B.SilkS) (width 0.12))
+    (fp_line (start -4.6 -6.9) (end -7.25 -6.9) (layer B.SilkS) (width 0.12))
+    (fp_line (start 8 -7.9) (end 8 3.2) (layer B.SilkS) (width 0.12))
+    (fp_line (start -8.05 3.2) (end 8 3.2) (layer B.SilkS) (width 0.12))
+    (fp_line (start 8 -2.45) (end 8 -7.9) (layer B.SilkS) (width 0.12))
+    (fp_line (start -8.05 -7.9) (end 8 -7.9) (layer B.SilkS) (width 0.12))
+    (fp_line (start -8.05 -7.9) (end -8.05 -6.9) (layer B.SilkS) (width 0.12))
+    (fp_line (start -8.05 -7.9) (end -8.05 3.2) (layer B.SilkS) (width 0.12))
+    (pad 1 thru_hole circle (at 5.9 -1.8 90) (size 1.524 1.524) (drill 0.762) (layers *.Cu *.Mask)
+      (net 9 "Net-(C6-Pad1)"))
+    (pad 2 thru_hole circle (at 5.9 0.9 90) (size 1.524 1.524) (drill 0.762) (layers *.Cu *.Mask)
+      (net 8 "Net-(R5-Pad1)"))
+  )
   (module Connector:FanPinHeader_1x03_P2.54mm_Vertical (layer F.Cu)
