File: mama_board/detector_circuit.kicad_pcb (KiCad board)
At the start: 4 copper layers, 94 x 99.1 mm, 124 parts, among them J1 Programming Header, J10 Conn_01x06_Female, J3 BATT_1, J4 BATT_2, J5 BATT_3, J6 BATT_4, J7 TEST_CONN, J8 693072010801, J9 SIPM_CONN, Q1 BSS138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

Commit message: Fixed some DRC issues
Routing:
- net GND: track 151.6 -> 138.0 mm
Other:
- rule pad_to_mask_clearance: 0 -> 0.0508
- rule solder_mask_min_width: 0.25 -> 0.101
Changed lines of the file:
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@@
     (thickness 1.6)
     (drawings 123)
-    (tracks 864)
+    (tracks 859)
     (zones 0)
     (modules 124)
@@
   )
   (setup
-    (last_trace_width 0.8)
+    (last_trace_width 1)
     (user_trace_width 0.42)
     (user_trace_width 0.8)
@@
     (pad_size 1.15 1.4)
     (pad_drill 0)
-    (pad_to_mask_clearance 0)
-    (solder_mask_min_width 0.25)
+    (pad_to_mask_clearance 0.0508)
+    (solder_mask_min_width 0.101)
     (aux_axis_origin 0 0)
     (grid_origin 151.765 64.135)
@@
   (segment (start 141.342 130.175) (end 139.827 130.175) (width 1) (layer Papa.Cu) (net 1))
   (via (at 144.399 124.841) (size 0.8) (drill 0.4) (layers Papa.Cu Mama.Cu) (net 1))
-  (via (at 101.981 96.647) (size 0.8) (drill 0.4) (layers Papa.Cu Mama.Cu) (net 1))
+  (via (at 98.298 96.647) (size 0.8) (drill 0.4) (layers Papa.Cu Mama.Cu) (net 1))
   (via (at 100.965 81.407) (size 0.8) (drill 0.4) (layers Papa.Cu Mama.Cu) (net 1))
   (via (at 101.854 76.073) (size 0.8) (drill 0.4) (layers Papa.Cu Mama.Cu) (net 1))
@@
   (segment (start 164.211 83.8835) (end 164.211 85.344) (width 1) (layer Papa.Cu) (net 1))
   (segment (start 155.693 83.7655) (end 153.797 85.6615) (width 1) (layer Papa.Cu) (net 1))
-  (segment (start 101.727 65.278) (end 101.092 65.913) (width 0.8) (layer Papa.Cu) (net 1))
-  (segment (start 95.211 65.913) (end 94.082 64.784) (width 0.8) (layer Papa.Cu) (net 1))
-  (segment (start 101.092 65.913) (end 95.211 65.913) (width 0.8) (layer Papa.Cu) (net 1))
-  (segment (start 101.727 59.182) (end 101.727 61.468) (width 0.8) (layer Papa.Cu) (net 1))
   (via (at 87.249 83.312) (size 0.8) (drill 0.4) (layers Papa.Cu Mama.Cu) (net 1))
   (via (at 162.941 130.556) (size 0.8) (drill 0.4) (layers Papa.Cu Mama.Cu) (net 1))
@@
   (segment (start 121.412 100.4205) (end 121.412 102.235) (width 1) (layer Papa.Cu) (net 1))
   (via (at 126.492 102.616) (size 0.8) (drill 0.4) (layers Papa.Cu Mama.Cu) (net 1))
-  (segment (start 101.727 61.468) (end 101.727 63.754) (width 0.8) (layer Papa.Cu) (net 1))
   (via (at 164.211 111.633) (size 0.8) (drill 0.4) (layers Papa.Cu Mama.Cu) (net 1))
   (segment (start 162.95 111.633) (end 164.211 111.633) (width 1) (layer Papa.Cu) (net 1))
@@
   (segment (start 124.215 64.5885) (end 124.206 64.5795) (width 1) (layer Papa.Cu) (net 1))
   (segment (start 124.215 66.548) (end 124.215 64.5885) (width 1) (layer Papa.Cu) (net 1))
-  (segment (start 101.727 63.754) (end 101.727 65.278) (width 0.8) (layer Papa.Cu) (net 1))
-  (via (at 101.727 63.754) (size 0.8) (drill 0.4) (layers Papa.Cu Mama.Cu) (net 1))
-  (segment (start 100.212 63.754) (end 101.727 63.754) (width 1) (layer Papa.Cu) (net 1))
+  (via (at 100.203 65.786) (size 0.8) (drill 0.4) (layers Papa.Cu Mama.Cu) (net 1))
   (segment (start 100.212 57.667) (end 100.203 57.658) (width 1) (layer Papa.Cu) (net 1))
   (segment (start 100.212 60.198) (end 100.212 57.667) (width 1) (layer Papa.Cu) (net 1))
   (segment (start 108.594 55.245) (end 111.379 55.245) (width 1) (layer Papa.Cu) (net 1))
-  (segment (start 101.972 96.656) (end 101.981 96.647) (width 1) (layer Papa.Cu) (net 1))
-  (segment (start 100.33 96.656) (end 101.972 96.656) (width 1) (layer Papa.Cu) (net 1))
   (segment (start 85.7885 100.5205) (end 85.7885 100.5205) (width 1) (layer Papa.Cu) (net 1))
   (via (at 85.7885 100.5205) (size 0.8) (drill 0.4) (layers Papa.Cu Mama.Cu) (net 1))
@@
   (segment (start 126.492 102.616) (end 126.492 100.4205) (width 1) (layer Papa.Cu) (net 1))
   (segment (start 152.4 114.681) (end 152.4 112.54) (width 1) (layer Papa.Cu) (net 1))
+  (segment (start 98.307 96.656) (end 98.298 96.647) (width 1) (layer Papa.Cu) (net 1))
+  (segment (start 100.33 96.656) (end 98.307 96.656) (width 1) (layer Papa.Cu) (net 1))
+  (segment (start 100.212 65.777) (end 100.203 65.786) (width 1) (layer Papa.Cu) (net 1))
+  (segment (start 100.212 63.754) (end 100.212 65.777) (width 1) (layer Papa.Cu) (net 1))
   (via (at 96.647 71.247) (size 0.8) (drill 0.4) (layers Papa.Cu Mama.Cu) (net 2))
   (via (at 98.171 57.531) (size 0.8) (drill 0.4) (layers Papa.Cu Mama.Cu) (net 2))
@@
     (polygon
       (pts
-        (xy 174.752 77.216) (xy 160.909 77.089) (xy 160.909 64.389) (xy 174.752 64.389)
+        (xy 174.752 77.216) (xy 170.688 77.216) (xy 170.688 73.914) (xy 165.354 73.914) (xy 165.227 77.126282)
+        (xy 160.909 77.089) (xy 161.00425 64.516) (xy 165.354 64.516) (xy 165.354 67.818) (xy 170.434 67.945)
+        (xy 170.434 64.516) (xy 174.6885 64.516)
       )
     )

Commit message: Added 2nd kind of transimpedance amplifier
Parts:
- removed G***: LOGO, Team_Logo:Logo_SilkScreen_15mm
- removed REF** (x4): MountingHole_3.5mm_Pad, MountingHole:MountingHole_3.5mm_Pad
- added C28: C, Capacitor_SMD:C_0805_2012Metric_Pad1.15x1.40mm_HandSolder, B.Cu at (111.3, 126.9)
- added C29: C, Capacitor_SMD:C_0805_2012Metric_Pad1.15x1.40mm_HandSolder, B.Cu at (107.7, 126.9)
- added C30: 0, Capacitor_SMD:C_0805_2012Metric_Pad1.15x1.40mm_HandSolder, B.Cu at (101.5, 135.0)
- added C34: 1n, Capacitor_SMD:C_0805_2012Metric_Pad1.15x1.40mm_HandSolder, B.Cu at (104.9, 134.9)
- added C38: C, Capacitor_SMD:C_0805_2012Metric_Pad1.15x1.40mm_HandSolder, B.Cu at (116.2, 136.8)
- added R43: 0, Resistor_SMD:R_0805_2012Metric_Pad1.15x1.40mm_HandSolder, B.Cu at (111.3, 131.1)
- added R44: 1k, Resistor_SMD:R_0805_2012Metric_Pad1.15x1.40mm_HandSolder, B.Cu at (107.7, 131.1)
- added R45: 0, Resistor_SMD:R_0805_2012Metric_Pad1.15x1.40mm_HandSolder, B.Cu at (98.0, 134.9)
- added R46: 1k, Resistor_SMD:R_0805_2012Metric_Pad1.15x1.40mm_HandSolder, B.Cu at (95.0, 134.9)
- added U7: LTC6269, Package_SO:MSOP-8_3x3mm_P0.65mm, B.Cu at (110.7, 135.4)
Connections:
- net Net-(C17-Pad2) renamed /Filter_IN
Routing:
- net /SIPM_OUT: track 29.5 -> 57.9 mm
- net /Filter_IN: track 17.7 -> 45.2 mm
- net +5V: track 81.6 -> 61.4 mm
- net Net-(C30-Pad2): track 0.00 -> 18.4 mm
- net GND: track 138.0 -> 154.1 mm, vias 125 -> 127
- net +4.7V: track 82.0 -> 87.4 mm, vias 6 -> 7
