File: mama_board/power_supplies.kicad_sch (KiCad schematic)
At the start: 12 parts, among them J7 TEST_CONN, U2 LD3985M47R_SOT23, U3 LT3014IS5#TRMPBF

Commit message: changed SD card resistors
Parts:
- R8: value 3.5k -> 3.330k
Other:
- note added: "SWAPPED FROM 3.5K NEED TO ORDER THSE"
Changed lines of the file:
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@@
     (effects (font (size 1.27 1.27)) (justify left bottom))
+  )
+  (text "SWAPPED FROM 3.5K NEED TO ORDER THSE" (at 161.29 137.16 270)
+    (effects (font (size 1.27 1.27)) (justify right bottom))
   )
   (global_label "+5.4V" (shape input) (at 124.46 58.42 180) (fields_autoplaced)
@@
       (effects (font (size 1.27 1.27)) (justify left))
     )
-    (property "Value" "3.5k" (id 1) (at 166.878 140.843 0)
+    (property "Value" "3.330k" (id 1) (at 166.878 140.843 0)
       (effects (font (size 1.27 1.27)) (justify left))
     )
