File: Papa_Board/payload2020_base_board.kicad_pcb (KiCad board)
At the start: 4 copper layers, 82 x 82 mm, 103 parts, among them J1 1862, J10 1862, J11 Conn_01x05, J2 Conn_01x05, J3 Conn_01x05_Female, J4 Conn_01x05, J5 M80-5000642, J6 M80-5000642, J7 1862, J8 693072010801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

Commit message: Clean up dimensions, add gerber zip file
Other:
- board text removed: "31.75 mm"
Changed lines of the file:
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@@
   (general
     (thickness 1.6)
-    (drawings 153)
+    (drawings 147)
     (tracks 1029)
     (zones 0)
@@
   (layers
     (0 F.Cu signal)
-    (1 GND.Cu power)
-    (2 VCC.Cu power)
-    (31 B.Cu signal)
-    (32 B.Adhes user)
-    (33 F.Adhes user)
-    (34 B.Paste user)
+    (1 GND.Cu power hide)
+    (2 VCC.Cu power hide)
+    (31 B.Cu signal hide)
+    (32 B.Adhes user hide)
+    (33 F.Adhes user hide)
+    (34 B.Paste user hide)
     (35 F.Paste user)
-    (36 B.SilkS user)
+    (36 B.SilkS user hide)
     (37 F.SilkS user)
-    (38 B.Mask user)
+    (38 B.Mask user hide)
     (39 F.Mask user)
     (40 Dwgs.User user)
-    (41 Cmts.User user)
-    (42 Eco1.User user)
-    (43 Eco2.User user)
+    (41 Cmts.User user hide)
+    (42 Eco1.User user hide)
+    (43 Eco2.User user hide)
     (44 Edge.Cuts user)
-    (45 Margin user)
-    (46 B.CrtYd user)
+    (45 Margin user hide)
+    (46 B.CrtYd user hide)
     (47 F.CrtYd user)
-    (48 B.Fab user)
+    (48 B.Fab user hide)
     (49 F.Fab user)
   )
@@
     (solder_mask_min_width 0.25)
     (aux_axis_origin 0 0)
-    (grid_origin 35.56 67.31)
+    (grid_origin 154.454 124.698)
     (visible_elements 7FFFF7FF)
     (pcbplotparams
@@
       (effects (font (size 1 1) (thickness 0.15)))
     )
-    (fp_circle (center 0 0) (end 3.5 0) (layer Cmts.User) (width 0.15))
     (fp_circle (center 0 0) (end 3.75 0) (layer F.CrtYd) (width 0.05))
+    (fp_circle (center 0 0) (end 3.5 0) (layer Cmts.User) (width 0.15))
     (pad 1 thru_hole circle (at 0 0) (size 7 7) (drill 3.5) (layers *.Cu *.Mask))
   )
@@
     )
   )
+  (gr_line (start 183.854 124.698) (end 154.454 124.698) (layer Dwgs.User) (width 0.15))
+  (gr_line (start 154.454 124.698) (end 154.454 67.818) (layer Dwgs.User) (width 0.15))
+  (dimension 31.75 (width 0.15) (layer Dwgs.User)
+    (gr_text "31.750 mm" (at 193.07 108.823) (layer Dwgs.User)
+      (effects (font (size 1 1) (thickness 0.15)) (justify left))
+    )
+    (feature1 (pts (xy 183.854 124.698) (xy 192.356421 124.698)))
+    (feature2 (pts (xy 183.854 92.948) (xy 192.356421 92.948)))
+    (crossbar (pts (xy 191.77 92.948) (xy 191.77 124.698)))
+    (arrow1a (pts (xy 191.77 124.698) (xy 191.183579 123.571496)))
+    (arrow1b (pts (xy 191.77 124.698) (xy 192.356421 123.571496)))
+    (arrow2a (pts (xy 191.77 92.948) (xy 191.183579 94.074504)))
+    (arrow2b (pts (xy 191.77 92.948) (xy 192.356421 94.074504)))
+  )
   (dimension 25.4 (width 0.15) (layer Dwgs.User)
     (gr_text "25.400 mm" (at 167.154 59.152) (layer Dwgs.User)
@@
   (gr_line (start 101.854 133.138) (end 129.794 133.1468) (layer Dwgs.User) (width 0.15))
   (dimension 48.64 (width 0.15) (layer Dwgs.User)
-    (gr_text "48.640 mm" (at 80.107 108.818 270) (layer Dwgs.User)
+    (gr_text "48.640 mm" (at 92.426 108.818) (layer Dwgs.User)
       (effects (font (size 1 1) (thickness 0.15)) (justify right))
     )
-    (feature1 (pts (xy 101.854 133.138) (xy 80.820579 133.138)))
-    (feature2 (pts (xy 101.854 84.498) (xy 80.820579 84.498)))
-    (crossbar (pts (xy 81.407 84.498) (xy 81.407 133.138)))
-    (arrow1a (pts (xy 81.407 133.138) (xy 80.820579 132.011496)))
-    (arrow1b (pts (xy 81.407 133.138) (xy 81.993421 132.011496)))
-    (arrow2a (pts (xy 81.407 84.498) (xy 80.820579 85.624504)))
-    (arrow2b (pts (xy 81.407 84.498) (xy 81.993421 85.624504)))
+    (feature1 (pts (xy 101.854 133.138) (xy 93.139579 133.138)))
+    (feature2 (pts (xy 101.854 84.498) (xy 93.139579 84.498)))
+    (crossbar (pts (xy 93.726 84.498) (xy 93.726 133.138)))
+    (arrow1a (pts (xy 93.726 133.138) (xy 93.139579 132.011496)))
+    (arrow1b (pts (xy 93.726 133.138) (xy 94.312421 132.011496)))
+    (arrow2a (pts (xy 93.726 84.498) (xy 93.139579 85.624504)))
+    (arrow2b (pts (xy 93.726 84.498) (xy 94.312421 85.624504)))
   )
   (dimension 12.68 (width 0.15) (layer Dwgs.User)
-    (gr_text "12.680 mm" (at 92.426 78.158 270) (layer Dwgs.User)
-      (effects (font (size 1 1) (thickness 0.15)))
+    (gr_text "12.680 mm" (at 92.426 78.158) (layer Dwgs.User)
+      (effects (font (size 1 1) (thickness 0.15)) (justify right))
     )
     (feature1 (pts (xy 105.854 84.498) (xy 93.139579 84.498)))
@@
     (arrow2b (pts (xy 93.726 71.818) (xy 94.312421 72.944504)))
   )
-  (gr_text "31.75 mm\n" (at 199.3392 110.744) (layer Dwgs.User)
-    (effects (font (size 1 1) (thickness 0.15)))
-  )
-  (gr_line (start 194.564 92.964) (end 195.2244 94.0816) (layer Dwgs.User) (width 0.15))
-  (gr_line (start 194.564 93.0148) (end 193.9036 94.0816) (layer Dwgs.User) (width 0.15))
-  (gr_line (start 194.564 124.6632) (end 195.2244 123.5964) (layer Dwgs.User) (width 0.15))
-  (gr_line (start 194.564 124.714) (end 193.9036 123.5964) (layer Dwgs.User) (width 0.15))
-  (gr_line (start 194.564 92.964) (end 194.564 124.714) (layer Dwgs.User) (width 0.15))
-  (gr_line (start 154.432 124.714) (end 195.15328 124.714) (layer Dwgs.User) (width 0.15))
-  (gr_line (start 191.77 92.948) (end 195.15328 92.94622) (layer Dwgs.User) (width 0.15))
-  (gr_line (start 179.854 92.948) (end 191.77 92.948) (layer Dwgs.User) (width 0.15))
   (dimension 21.13 (width 0.15) (layer Dwgs.User)
     (gr_text "21.130 mm" (at 193.07 82.383) (layer Dwgs.User)
@@
   )
   (dimension 4.000496 (width 0.15) (layer Dwgs.User)
-    (gr_text "4.000 mm" (at 95.932379 147.662231 89.09766608) (layer Dwgs.User)
-      (effects (font (size 1 1) (thickness 0.15)))
+    (gr_text "4.000 mm" (at 95.932379 147.662231) (layer Dwgs.User)
+      (effects (font (size 1 1) (thickness 0.15)) (justify right))
     )
     (feature1 (pts (xy 105.791 149.818) (xy 96.61437 149.673468)))
@@
   )
   (dimension 4 (width 0.15) (layer Dwgs.User)
-    (gr_text "4.000 mm" (at 190.954 147.818) (layer Dwgs.User)
+    (gr_text "4.000 mm" (at 193.536 147.818) (layer Dwgs.User)
       (effects (font (size 1 1) (thickness 0.15)) (justify left))
     )
-    (feature1 (pts (xy 179.854 145.818) (xy 190.240421 145.818)))
-    (feature2 (pts (xy 179.854 149.818) (xy 190.240421 149.818)))
-    (crossbar (pts (xy 189.654 149.818) (xy 189.654 145.818)))
-    (arrow1a (pts (xy 189.654 145.818) (xy 190.240421 146.944504)))
-    (arrow1b (pts (xy 189.654 145.818) (xy 189.067579 146.944504)))
-    (arrow2a (pts (xy 189.654 149.818) (xy 190.240421 148.691496)))
-    (arrow2b (pts (xy 189.654 149.818) (xy 189.067579 148.691496)))
+    (feature1 (pts (xy 179.854 145.818) (xy 192.822421 145.818)))
+    (feature2 (pts (xy 179.854 149.818) (xy 192.822421 149.818)))
+    (crossbar (pts (xy 192.236 149.818) (xy 192.236 145.818)))
+    (arrow1a (pts (xy 192.236 145.818) (xy 192.822421 146.944504)))
+    (arrow1b (pts (xy 192.236 145.818) (xy 191.649579 146.944504)))
+    (arrow2a (pts (xy 192.236 149.818) (xy 192.822421 148.691496)))
+    (arrow2b (pts (xy 192.236 149.818) (xy 191.649579 148.691496)))
   )
   (dimension 4.00006 (width 0.15) (layer Dwgs.User)
-    (gr_text "4.000 mm" (at 103.7869 158.006917 359.6848764) (layer Dwgs.User)
+    (gr_text "4.000 mm" (at 103.7869 158.006917) (layer Dwgs.User)
       (effects (font (size 1 1) (thickness 0.15)))
     )
@@
   (dimension 5 (width 0.15) (layer Dwgs.User)
     (gr_text "5.000 mm" (at 142.718 147.318) (layer Dwgs.User)
-      (effects (font (size 1 1) (thickness 0.15)))
+      (effects (font (size 1 1) (thickness 0.15)) (justify right))
     )
     (feature1 (pts (xy 150.354 149.818) (xy 143.431579 149.818)))
@@
   )
   (dimension 15 (width 0.15) (layer Dwgs.User)
-    (gr_text "15.000 mm" (at 142.854 162.59) (layer Dwgs.User)
+    (gr_text "15.000 mm" (at 142.854 158.78) (layer Dwgs.User)
       (effects (font (size 1 1) (thickness 0.15)))
     )
-    (feature1 (pts (xy 150.354 149.818) (xy 150.354 161.876421)))
-    (feature2 (pts (xy 135.354 149.818) (xy 135.354 161.876421)))
-    (crossbar (pts (xy 135.354 161.29) (xy 150.354 161.29)))
-    (arrow1a (pts (xy 150.354 161.29) (xy 149.227496 161.876421)))
-    (arrow1b (pts (xy 150.354 161.29) (xy 149.227496 160.703579)))
-    (arrow2a (pts (xy 135.354 161.29) (xy 136.480504 161.876421)))
-    (arrow2b (pts (xy 135.354 161.29) (xy 136.480504 160.703579)))
+    (feature1 (pts (xy 150.354 149.818) (xy 150.354 158.066421)))
+    (feature2 (pts (xy 135.354 149.818) (xy 135.354 158.066421)))
+    (crossbar (pts (xy 135.354 157.48) (xy 150.354 157.48)))
+    (arrow1a (pts (xy 150.354 157.48) (xy 149.227496 158.066421)))
+    (arrow1b (pts (xy 150.354 157.48) (xy 149.227496 156.893579)))
+    (arrow2a (pts (xy 135.354 157.48) (xy 136.480504 158.066421)))
+    (arrow2b (pts (xy 135.354 157.48) (xy 136.480504 156.893579)))
   )
   (dimension 82 (width 0.15) (layer Dwgs.User)
@@
   )
   (dimension 82 (width 0.15) (layer Dwgs.User)
-    (gr_text "82.000 mm" (at 207.294 108.818 270) (layer Dwgs.User)
-      (effects (font (size 1 1) (thickness 0.15)))
+    (gr_text "82.000 mm" (at 207.294 108.818) (layer Dwgs.User)
+      (effects (font (size 1 1) (thickness 0.15)) (justify left))
     )
     (feature1 (pts (xy 183.854 149.818) (xy 206.580421 149.818)))
