File: Papa_Board/pic_and_can_controllers.kicad_sch (KiCad schematic)
At the start: 29 parts, among them U10 MCP2562-E/SN, U5 MCP2515-I/P, U7 MCP2562-E/SN, U8 DSPIC33EP512GP502, Y1 12MHz, Y2 12MHz

Commit message: fixed volgtage logic levels, added test connectors and jumpers
Parts:
- removed C1, C2: 27pF, Capacitor_SMD:C_0805_2012Metric_Pad1.18x1.45mm_HandSolder, symbol Device:C_Small
- removed Y2: 12MHz, Crystal:Crystal_HC49-4H_Vertical, symbol Device:Crystal
- C11, C29: value 10uF -> 0.1uF
Connections:
- net OSC4 is gone; now on net CLKOUT: U5.8 (OSC1)
- net +3V3: now also C12.1, C14.1, C16.1, R2.1, R24.1, U10.5 (Vio), U5.18 (VDD), U7.5 (Vio)
- net +5V: no longer C12.1, C14.1, C16.1, R2.1, R24.1, U10.5 (Vio), U5.18 (VDD), U7.5 (Vio)
- net CLKOUT: no longer U5.3 (CLKOUT)
- net OSC3: no longer names the net of U5.7 (OSC2)
- no-connect marks 5 -> 7

Commit message: Address Jack's schematic review, still need to update PCB layout and figure out CAN connections
Parts:
- R4, R5, R9: value 500R -> 150R
- U8: value DSPIC33EP512GP502 -> DSPIC33EP256GP502
Other:
- note added: "Debugging LEDs Vs = 3.3V"
- note removed: "Debugging LEDs Vs = 5V"
Changed lines of the file:
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@@
     (effects (font (size 1.27 1.27)) (justify left bottom))
   )
-  (text "Debugging LEDs\nVs = 5V\n" (at 160.02 162.56 0)
+  (text "Debugging LEDs\nVs = 3.3V\n" (at 160.02 162.56 0)
     (effects (font (size 1.27 1.27)) (justify left bottom))
   )
@@
       (effects (font (size 1.27 1.27)) (justify left))
     )
-    (property "Value" "500R" (id 1) (at 166.8272 138.303 0)
+    (property "Value" "150R" (id 1) (at 166.8272 138.303 0)
       (effects (font (size 1.27 1.27)) (justify left))
     )
@@
       (effects (font (size 1.27 1.27)) (justify left))
     )
-    (property "Value" "500R" (id 1) (at 187.1472 135.763 0)
+    (property "Value" "150R" (id 1) (at 187.1472 135.763 0)
       (effects (font (size 1.27 1.27)) (justify left))
     )
@@
       (effects (font (size 1.27 1.27)) (justify left))
     )
-    (property "Value" "500R" (id 1) (at 150.3172 144.653 0)
+    (property "Value" "150R" (id 1) (at 150.3172 144.653 0)
       (effects (font (size 1.27 1.27)) (justify left))
     )
@@
     (in_bom yes) (on_board yes)
     (property "Reference" "U8" (id 0) (at 120.65 85.09 0))
-    (property "Value" "DSPIC33EP512GP502" (id 1) (at 120.65 87.63 0))
+    (property "Value" "DSPIC33EP256GP502" (id 1) (at 120.65 87.63 0))
     (property "Footprint" "Package_SO:SOIC-28W_7.5x17.9mm_P1.27mm" (id 2) (at 88.9 116.84 0)
       (effects (font (size 1.27 1.27)) hide)
