File: Papa_Board/battery_management.kicad_sch (KiCad schematic)
At the start: 53 parts, among them J1 Conn_01x02_Female, J10 Conn_01x02_Female, J11 GND TEST CONN, J7 Conn_01x02_Female, J9 Conn_01x02_Female, U1 INA180A4QDBVRQ1, U2 INA180A4QDBVRQ1, U3 AP1509, U4 FPF2125, U6 TPS61175QPWPRQ1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

Commit message: Address Zach + Jacks review, move mounting holes to fit logger, update pdf
Parts:
- U6: footprint Payload2020_custom:TPS61175_Q1_Footprint -> Package_SO:HTSSOP-14-1EP_4.4x5mm_P0.65mm_EP3.4x5mm_Mask3x3.1mm_ThermalVias
Changed lines of the file:
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@@
   (junction (at 29.972 59.69) (diameter 0) (color 0 0 0 0)
   )
+  (junction (at 41.91 104.14) (diameter 0) (color 0 0 0 0)
+  )
   (junction (at 194.818 50.8) (diameter 0) (color 0 0 0 0)
   )
@@
   (junction (at 78.74 43.18) (diameter 0) (color 0 0 0 0)
   )
-  (junction (at 51.308 111.76) (diameter 0) (color 0 0 0 0)
-  )
   (junction (at 58.42 189.23) (diameter 0) (color 0 0 0 0)
   )
@@
     (stroke (width 0) (type default) (color 0 0 0 0))
   )
+  (wire (pts (xy 50.8 111.76) (xy 51.308 111.76))
+    (stroke (width 0) (type default) (color 0 0 0 0))
+  )
   (wire (pts (xy 58.928 118.11) (xy 58.928 120.65))
     (stroke (width 0) (type default) (color 0 0 0 0))
@@
     (stroke (width 0) (type default) (color 0 0 0 0))
   )
-  (wire (pts (xy 51.435 111.76) (xy 51.308 111.76))
-    (stroke (width 0) (type default) (color 0 0 0 0))
-  )
   (wire (pts (xy 78.74 40.64) (xy 78.74 43.18))
     (stroke (width 0) (type default) (color 0 0 0 0))
   )
+  (wire (pts (xy 41.91 104.14) (xy 44.45 104.14))
+    (stroke (width 0) (type default) (color 0 0 0 0))
+  )
   (wire (pts (xy 62.23 152.4) (xy 67.31 152.4))
     (stroke (width 0) (type default) (color 0 0 0 0))
@@
     (stroke (width 0) (type default) (color 0 0 0 0))
   )
-  (wire (pts (xy 51.308 111.76) (xy 50.8 111.76))
-    (stroke (width 0) (type default) (color 0 0 0 0))
-  )
   (wire (pts (xy 160.02 40.64) (xy 167.64 40.64))
     (stroke (width 0) (type default) (color 0 0 0 0))
@@
     (stroke (width 0) (type default) (color 0 0 0 0))
   )
-  (wire (pts (xy 38.1 104.14) (xy 44.45 104.14))
+  (wire (pts (xy 38.1 104.14) (xy 41.91 104.14))
     (stroke (width 0) (type default) (color 0 0 0 0))
   )
@@
     (property "Reference" "U6" (id 0) (at 57.15 154.94 0))
     (property "Value" "TPS61175QPWPRQ1" (id 1) (at 57.15 157.48 0))
-    (property "Footprint" "Payload2020_custom:TPS61175_Q1_Footprint" (id 2) (at 57.15 168.91 0)
+    (property "Footprint" "Package_SO:HTSSOP-14-1EP_4.4x5mm_P0.65mm_EP3.4x5mm_Mask3x3.1mm_ThermalVias" (id 2) (at 57.15 168.91 0)
       (effects (font (size 1.27 1.27)) hide)
     )
@@
       (effects (font (size 1.27 1.27)) hide)
     )
+    (pin "1")
+  )
+  (symbol (lib_id "power:PWR_FLAG") (at 41.91 104.14 0) (unit 1)
+    (in_bom yes) (on_board yes) (fields_autoplaced)
+    (property "Reference" "#FLG0105" (id 0) (at 41.91 102.235 0)
+      (effects (font (size 1.27 1.27)) hide)
+    )
+    (property "Value" "PWR_FLAG" (id 1) (at 41.91 99.06 0))
+    (property "Footprint" "" (id 2) (at 41.91 104.14 0)
+      (effects (font (size 1.27 1.27)) hide)
+    )
+    (property "Datasheet" "~" (id 3) (at 41.91 104.14 0)
+      (effects (font (size 1.27 1.27)) hide)
+    )

Commit message: made last fixes & revision, generated gerbers
Other:
- note added: "1A max i think"
- note added: "Logic High"
Changed lines of the file:
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@@
+    (effects (font (size 1.27 1.27)) (justify left bottom))
+  )
+  (text "1A max i think " (at 177.8 134.62 0)
     (effects (font (size 1.27 1.27)) (justify left bottom))
   )
@@
     (effects (font (size 1.27 1.27)) (justify left bottom))
   )
+  (text "Logic High" (at 177.8 132.08 0)
+    (effects (font (size 1.27 1.27)) (justify left bottom))
+  )

Commit message: Update L2 footprint, silkscreen adjustments
Parts:
- L2: footprint Inductor_THT:L_Radial_D8.7mm_P5.00mm_Fastron_07HCP -> Inductor_SMD:L_Wuerth_WE-PD-Typ-LS_Handsoldering
Changed lines of the file:
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@@
     (property "Reference" "L2" (id 0) (at 95.758 97.79 0))
     (property "Value" "47uH" (id 1) (at 95.758 100.33 0))
-    (property "Footprint" "Inductor_THT:L_Radial_D8.7mm_P5.00mm_Fastron_07HCP" (id 2) (at 95.758 104.14 0)
+    (property "Footprint" "Inductor_SMD:L_Wuerth_WE-PD-Typ-LS_Handsoldering" (id 2) (at 95.758 104.14 0)
       (effects (font (size 1.27 1.27)) hide)
     )
